Commit message: New Robot implemented

File: catkin_ws/src/my_robot/urdf/my_robot.xacro (robot description, xacro)
@@ -15,8 +15,8 @@
       />
     </inertial>
-    <collision name='collision'>
-      <origin xyz="0 0 0" rpy=" 0 0 0"/>
-      <geometry>
-        <box size=".4 .2 .1"/>
+    <collision name='chassis_collision'>
+      <origin xyz="0 0 0" rpy=" 0 0 0"/>
+      <geometry>
+        <box size=".4 .3 .1"/>
       </geometry>
     </collision>
@@ -24,5 +24,5 @@
       <origin xyz="0 0 0" rpy=" 0 0 0"/>
       <geometry>
-        <box size=".4 .2 .1"/>
+        <box size=".4 .3 .1"/>
       </geometry>
     </visual>
@@ -49,4 +49,89 @@
       <geometry>
         <sphere radius="0.05"/>
+      </geometry>
+    </visual>
+    <!--Upper part of the body-->
+    <collision name='body_collision'>
+      <origin xyz="0 0 0.15" rpy=" 0 0 0"/>
+      <geometry>
+        <cylinder radius="0.14" length="0.2"/>
+      </geometry>
+    </collision>
+    <visual name='body_visual'>
+      <origin xyz="0 0 0.15" rpy=" 0 0 0"/>
+      <geometry>
+        <cylinder radius="0.14" length="0.2"/>
+      </geometry>
+    </visual>
+    <collision name='arm_rigth_collision'>
+      <origin xyz="0 -0.16 0.2" rpy=" 0 0 0"/>
+      <geometry>
+        <sphere radius="0.025"/>
+      </geometry>
+    </collision>
+    <visual name='arm_rigth_visual'>
+      <origin xyz="0 -0.16 0.2" rpy=" 0 0 0"/>
+      <geometry>
+        <sphere radius="0.025"/>
+      </geometry>
+    </visual>
+    <collision name='arm_R_collision'>
+      <origin xyz="0.03 -0.16 0.165" rpy=" 0 -0.6981 0"/>
+      <geometry>
+        <cylinder radius="0.025" length="0.1"/>
+      </geometry>
+    </collision>
+    <visual name='arm_R_visual'>
+      <origin xyz="0.03 -0.16 0.165" rpy=" 0 -0.6981 0"/>
+      <geometry>
+        <cylinder radius="0.025" length="0.1"/>
+      </geometry>
+    </visual>
+    <collision name='arm_left_collision'>
+      <origin xyz="0 0.16 0.2" rpy=" 0 0 0"/>
+      <geometry>
+        <sphere radius="0.025"/>
+      </geometry>
+    </collision>
+    <visual name='arm_left_visual'>
+      <origin xyz="0 0.16 0.2" rpy=" 0 0 0"/>
+      <geometry>
+        <sphere radius="0.025"/>
+      </geometry>
+    </visual>
+    <collision name='arm_L_collision'>
+      <origin xyz="0.03 0.16 0.165" rpy=" 0 -0.6981 0"/>
+      <geometry>
+        <cylinder radius="0.025" length="0.1"/>
+      </geometry>
+    </collision>
+    <visual name='arm_L_visual'>
+      <origin xyz="0.03 0.16 0.165" rpy=" 0 -0.6981 0"/>
+      <geometry>
+        <cylinder radius="0.025" length="0.1"/>
+      </geometry>
+    </visual>
+    <collision name='neck_collision'>
+      <origin xyz="-0.03 0 0.3" rpy=" 0 0 0"/>
+      <geometry>
+        <cylinder radius="0.03" length="0.1"/>
+      </geometry>
+    </collision>
+    <visual name='neck_visual'>
+      <origin xyz="-0.03 0 0.3" rpy=" 0 0 0"/>
+      <geometry>
+        <cylinder radius="0.03" length="0.1"/>
+      </geometry>
+    </visual>
+    <collision name='head_collision'>
+      <origin xyz="0 0 0.38" rpy=" 0 0.4363 0"/>
+      <geometry>
+        <cylinder radius="0.14" length="0.1"/>
+      </geometry>
+    </collision>
+    <visual name='head_visual'>
+      <origin xyz="0 0 0.38" rpy=" 0 0.4363 0"/>
+      <geometry>
+        <cylinder radius="0.14" length="0.1"/>
       </geometry>
     </visual>
@@ -156,5 +241,5 @@
   <!--Joints Wheels-->
   <joint type="continuous" name="left_wheel_hinge">
-    <origin xyz="0 0.15 0" rpy="0 0 0"/>
+    <origin xyz="0 0.18 0" rpy="0 0 0"/>
     <child link="left_wheel"/>
     <parent link="chassis"/>
@@ -164,5 +249,5 @@
   </joint>
   <joint type="continuous" name="right_wheel_hinge">
-    <origin xyz="0 -0.15 0" rpy="0 0 0"/>
+    <origin xyz="0 -0.18 0" rpy="0 0 0"/>
     <child link="right_wheel"/>
     <parent link="chassis"/>
@@ -180,5 +265,5 @@
   <!--Joint Hokuyo-->
   <joint type="fixed" name="hokuyo_joint">
-    <origin xyz="0.15 0 0.1" rpy="0 0 0"/>
+    <origin xyz="0.17 0 0.08" rpy="0 0 0"/>
     <child link="hokuyo"/>
     <parent link="chassis"/>
@@ -198,3 +283,6 @@
     <material>Gazebo/Blue</material>
   </gazebo>
+  <gazebo reference="body">
+    <material>Gazebo/Orange</material>
+  </gazebo>
 </robot>
